File: 月光2/月光2.kicad_pcb (KiCad board)
At the start: 2 copper layers, 40 x 60.5 mm, 73 parts, among them J1 Conn_01x12, J2 Conn_01x12, J3 Conn_01x05, J4 Conn_01x03, J6 Conn_01x02, Q1 Q_Photo_NPN, Q2 Q_Photo_NPN, Q3 Q_Photo_NPN, Q4 Q_Photo_NPN, Q5 IRLML6344TRPBFTR, SW1 SW_Push_Dual_x2, U1 DRV8835, U2 STM32F413CH6, U4 LP5907_DBV, U5 ICM20648, Y1 Crystal_GND23

Commit message: haisenmae
Parts:
- moved RN1 12.2 mm to (144.3, 118.3), turned to 270 degrees
- moved RN2 11.3 mm to (155.0, 122.8), turned to 270 degrees
- moved R26 9.53 mm to (138.8, 106.2), turned to 270 degrees
- moved R4 9.43 mm to (161.4, 106.2), turned to 90 degrees
- moved C25 8.76 mm to (130.9, 137.4), turned to 90 degrees
- moved R22 7.62 mm to (157.7, 101.2), turned to 40 degrees
- moved R28 7.36 mm to (142.9, 100.8), turned to 140 degrees
- moved R23 7.22 mm to (137.5, 106.2), turned to 90 degrees
- moved R5 7.16 mm to (162.6, 106.2), turned to 270 degrees
- moved C1 7.10 mm to (137.3, 138.5), turned to 90 degrees
- moved R21 6.93 mm to (142.1, 101.7), turned to 140 degrees
- moved C26 6.91 mm to (137.3, 135.2), turned to 90 degrees
- moved R27 6.78 mm to (156.9, 100.3), turned to 40 degrees
- moved R3 5.99 mm to (137.5, 103.8)
- moved U4 5.52 mm to (134.2, 136.7)
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Other:
- outline, holes or cut-outs redrawn

Commit message: #
Parts:
- moved R27 1.37 mm to (155.6, 100.9)
- moved C20 1.03 mm to (139.3, 98.8)
- moved C21 0.56 mm to (160.6, 98.5)
- moved R22 0.36 mm to (157.3, 101.3)
- moved D2 0.24 mm to (135.3, 108.9)
- moved Q1 0.20 mm to (135.5, 111.2)
- moved D3 0.16 mm to (154.8, 98.4)
- moved Q3 0.16 mm to (153.1, 99.9)

Commit message: #
Parts:
- D1, D3, Q2, Q3: footprint LED_THT:LED_D3.0mm_Horizontal_O3.81mm_Z2.0mm -> micro:micro_reverce_LED
- moved R6 19.0 mm to (157.0, 117.5)
- moved C11 6.16 mm to (144.0, 102.1), turned to 90 degrees
- moved R21 4.89 mm to (140.2, 106.2), turned to 90 degrees
- moved R28 3.95 mm to (140.3, 103.8), turned to 90 degrees
- moved R27 0.74 mm to (156.2, 100.4)
- moved C10 0.41 mm to (149.9, 100.0)
- moved R2 0.15 mm to (138.9, 103.8)
- moved R26 0.12 mm to (138.9, 106.2)
- turned C6 to 270 degrees
- turned L1 to 0 degrees
Routing:
- net CS_IMU: track 0.00 -> 22.0 mm, vias 0 -> 2
- net +3V3: track 0.00 -> 9.75 mm
- net GND: track 0.00 -> 6.75 mm
- net Net-(C6-Pad2): track 0.00 -> 4.80 mm
- net SCK_IMU: track 0.00 -> 4.69 mm, vias 0 -> 1
- net Net-(C11-Pad1): track 0.00 -> 3.50 mm
- net MOSI_IMU: track 0.00 -> 3.46 mm, vias 0 -> 1
- net Net-(C10-Pad1): track 0.00 -> 3.07 mm
- net CROCK_IN: track 0.00 -> 2.82 mm

Commit message: ##
Parts:
- moved R3 26.1 mm to (163.3, 100.3)
- moved R16 13.7 mm to (157.1, 123.3)
- moved R28 11.8 mm to (148.6, 95.4), turned to 315 degrees
- moved RN1 11.5 mm to (155.9, 118.1)
- moved RN2 10.7 mm to (144.3, 122.7)
- moved R18 9.90 mm to (149.9, 145.3), turned to 0 degrees
- moved R20 8.43 mm to (153.4, 123.4)
- moved D8 7.01 mm to (149.9, 137.7), turned to 180 degrees
- moved R23 5.37 mm to (141.5, 102.6), turned to 270 degrees
- moved D10 4.77 mm to (149.9, 146.6), turned to 180 degrees
- moved R14 4.36 mm to (149.9, 144.0), turned to 0 degrees
- moved R6 3.86 mm to (153.1, 117.4)
- moved D7 3.29 mm to (149.9, 142.7), turned to 180 degrees
- moved R10 2.67 mm to (149.9, 140.2), turned to 180 degrees
- moved D5 2.43 mm to (149.9, 141.5), turned to 180 degrees
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Routing:
- net encL_2: track 0.00 -> 56.8 mm, vias 0 -> 2
- net UART_TX: track 0.00 -> 55.0 mm, vias 0 -> 2
- net NRST: track 0.00 -> 52.8 mm, vias 0 -> 2
- net UART_RX: track 0.00 -> 49.9 mm, vias 0 -> 2
- net encR_1: track 0.00 -> 47.8 mm, vias 0 -> 2
- net STLINK_TCK: track 0.00 -> 47.6 mm, vias 0 -> 4
- net encL_1: track 0.00 -> 42.2 mm, vias 0 -> 2
- net MISO_IMU: track 0.00 -> 41.1 mm, vias 0 -> 3
- net encR_2: track 0.00 -> 37.0 mm, vias 0 -> 2
- net SCK_IMU: track 4.69 -> 25.7 mm, vias 1 -> 4
- net MOSI_IMU: track 3.46 -> 22.3 mm, vias 1 -> 2
- net +3V3: track 9.75 -> 26.7 mm, vias 0 -> 2
- net MORTOR_2+: track 0.00 -> 16.3 mm
- net MORTOR_2-: track 0.00 -> 15.7 mm
- net MORTOR_1-: track 0.00 -> 13.2 mm
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
Commit message: finish
Parts:
- moved R3 21.3 mm to (142.1, 101.9), turned to 180 degrees
- moved Q5 20.1 mm to (143.0, 104.4)
- moved R23 9.93 mm to (148.9, 96.0), turned to 315 degrees
- moved C21 9.90 mm to (153.4, 91.7)
- moved C19 9.65 mm to (160.9, 98.1)
- moved R16 8.67 mm to (157.2, 132.0)
- moved R22 8.34 mm to (151.2, 95.7), turned to 45 degrees
- moved R27 8.21 mm to (150.3, 94.7), turned to 225 degrees
- moved R4 4.22 mm to (161.3, 102.0), turned to 270 degrees
- moved C4 2.75 mm to (147.0, 134.8)
- moved R21 2.06 mm to (138.3, 105.3), turned to 180 degrees
- moved R28 1.85 mm to (149.4, 93.7), turned to 225 degrees
- moved R5 1.70 mm to (161.6, 104.9)
- moved U1 1.67 mm to (149.9, 134.3)
- moved R2 1.18 mm to (137.6, 103.3)
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Connections:
- U2 pad 42: MotorR_Foward -> MotorR_Reverce
- U2 pad 43: MotorR_Reverce -> MotorR_Foward
Routing:
- net GND: track 18.3 -> 247.9 mm, vias 0 -> 25
- net +3V3: track 26.7 -> 183.2 mm, vias 2 -> 21
- net sens_RR: track 0.00 -> 52.9 mm, vias 0 -> 4
- net STLINK_TMS: track 5.30 -> 58.2 mm, vias 1 -> 4
- net +BATT: track 3.88 -> 55.6 mm, vias 0 -> 5
- net Net-(D1-Pad1): track 0.00 -> 48.4 mm, vias 0 -> 7
- net sens_R: track 0.00 -> 41.1 mm, vias 0 -> 3
- net MotorL_Foward: track 0.00 -> 36.2 mm, vias 0 -> 4
- net MotorL_Reverce: track 0.00 -> 35.1 mm, vias 0 -> 4
- net MotorR_Foward: track 0.00 -> 29.3 mm, vias 0 -> 2
- net MotorR_Reverce: track 0.00 -> 28.8 mm, vias 0 -> 2
- net sens_LL: track 0.00 -> 21.7 mm, vias 0 -> 2
- net sens_L: track 0.00 -> 20.6 mm, vias 0 -> 2
- net RLED_PWM: track 0.00 -> 18.2 mm, vias 0 -> 2
- net Net-(D9-Pad2): track 0.00 -> 15.6 mm, vias 0 -> 2
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
Commit message: finish 2
Routing:
- net +3V3: track 183.2 -> 198.6 mm, vias 21 -> 25
- net NRST: track 59.7 -> 57.3 mm
- net STLINK_TCK: track 48.3 -> 49.1 mm

Commit message: finish 3
Parts:
- removed D1, D3: LED, micro:micro_reverce_LED
- removed D2, D4: LED, LED_THT:LED_D3.0mm_Horizontal_O3.81mm_Z2.0mm
- removed Q1, Q4: Q_Photo_NPN, LED_THT:LED_D3.0mm_Horizontal_O3.81mm_Z2.0mm
- removed Q2, Q3: Q_Photo_NPN, micro:micro_reverce_LED
- added U3: LED_FOTR, micro:LED_FOTR, F.Cu at (133.1, 110.9)
- added U6: LED_FOTR, micro:LED_FOTR, F.Cu at (146.7, 99.8)
- added U7: LED_FOTR, micro:LED_FOTR_M, F.Cu at (151.5, 97.8)
- added U8: LED_FOTR, micro:LED_FOTR_M, F.Cu at (164.4, 110.7)
- moved R24 1.25 mm to (149.2, 89.0)
- moved R8 1.13 mm to (148.1, 89.0)
- moved R23 0.71 mm to (148.7, 95.3)
- moved J4 0.28 mm to (166.6, 135.9)
- moved R25 0.14 mm to (151.7, 89.0)
- moved R7 0.07 mm to (150.5, 88.9)
Connections:
- R24 pad 1: sens_LL -> sens_R
- R25 pad 1: sens_RR -> sens_LL
- R7 pad 1: sens_R -> sens_RR
- U2 pad 13: sens_RR -> sens_LL
- U2 pad 14: sens_R -> sens_RR
- U2 pad 15: sens_L -> sens_R
- U2 pad 16: sens_LL -> sens_L
Routing:
- net LED_3: track 0.00 -> 60.0 mm, vias 0 -> 4
- net LED_1: track 0.00 -> 50.8 mm, vias 0 -> 2
- net LED_2: track 0.00 -> 45.9 mm, vias 0 -> 4
- net sens_LL: track 21.7 -> 52.5 mm, vias 2 -> 4
- net sens_R: track 41.1 -> 20.5 mm, vias 3 -> 2
- net sens_RR: track 52.9 -> 41.1 mm, vias 4 -> 3
- net GND: track 247.9 -> 258.4 mm, vias 25 -> 23
- net STLINK_TMS: track 58.2 -> 50.4 mm, vias 4 -> 5
- net +3V3: track 198.6 -> 192.4 mm
- net STLINK_TCK: track 49.1 -> 44.1 mm
- net NRST: track 57.3 -> 53.5 mm
- net UART_TX: track 56.1 -> 53.4 mm
- net RLED_PWM: track 18.2 -> 16.5 mm
- net sens_L: track 20.6 -> 21.8 mm
- net Net-(C22-Pad1): track 4.32 -> 3.47 mm
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
Commit message: finish 4
Routing:
- net GND: track 258.4 -> 273.3 mm, vias 23 -> 25
- net +3V3: track 192.4 -> 198.2 mm
- net STLINK_TMS: track 50.4 -> 56.1 mm, vias 5 -> 6
- net STLINK_TCK: track 44.1 -> 48.9 mm
- net NRST: track 53.5 -> 57.2 mm
- net UART_TX: track 53.4 -> 56.2 mm
Changed lines of the file:
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@@
     (thickness 1.6)
     (drawings 82)
-    (tracks 1238)
+    (tracks 1272)
     (zones 0)
     (modules 69)
@@
   )
   (module micro:LED_FOTR_M (layer F.Cu)
-    (at 151.5 97.82 310)
+    (at 151.48 97.82 310)
     (fp_text reference U7 (at -9.4 -0.4 130) (layer F.SilkS)
       (effects (font (size 1 1) (thickness 0.1)))
@@
   (via (at 167.06 133.82) (size 0.6) (drill 0.3) (layers F.Cu B.Cu) (net 1))
   (segment (start 167.06 133.82) (end 163.208559 137.671441) (width 0.2) (layer B.Cu) (net 1))
+  (segment (start 163.45 141.61) (end 163.87 141.61) (width 0.2) (layer F.Cu) (net 1))
+  (segment (start 167.28 145.02) (end 167.89 145.02) (width 0.2) (layer F.Cu) (net 1))
+  (segment (start 163.87 141.61) (end 167.28 145.02) (width 0.2) (layer F.Cu) (net 1))
   (segment (start 161.96999 141.99999) (end 161.93 141.96) (width 0.2) (layer F.Cu) (net 2))
   (segment (start 150.44 122.435) (end 151.24 123.235) (width 0.2) (layer F.Cu) (net 2))
@@
   (segment (start 164.82 131.39) (end 165.38999 131.95999) (width 0.2) (layer F.Cu) (net 2))
   (segment (start 168.339999 143.139999) (end 168.31 143.11) (width 0.2) (layer F.Cu) (net 2))
-  (segment (start 163.39 142.53) (end 163.39 143.66) (width 0.2) (layer F.Cu) (net 2))
   (segment (start 162.6 141.95) (end 163.3 142.65) (width 0.2) (layer F.Cu) (net 2))
   (segment (start 162.1 141.95) (end 162.6 141.95) (width 0.2) (layer F.Cu) (net 2))
@@
   (segment (start 165.38999 131.95999) (end 165.38999 134.08999) (width 0.2) (layer F.Cu) (net 2))
   (segment (start 165.38999 134.08999) (end 167.6 136.3) (width 0.2) (layer F.Cu) (net 2))
-  (segment (start 167.6 136.3) (end 167.6 137.67) (width 0.2) (layer F.Cu) (net 2))
+  (segment (start 163.630001 143.480001) (end 163.93 143.78) (width 0.2) (layer F.Cu) (net 2))
+  (via (at 163.93 143.78) (size 0.6) (drill 0.3) (layers F.Cu B.Cu) (net 2))
+  (segment (start 163.56 142.5) (end 163.56 143.41) (width 0.2) (layer F.Cu) (net 2))
+  (segment (start 163.56 143.41) (end 163.630001 143.480001) (width 0.2) (layer F.Cu) (net 2))
+  (via (at 166.16 142.14) (size 0.6) (drill 0.3) (layers F.Cu B.Cu) (net 2))
+  (segment (start 164.52 143.78) (end 165.860001 142.439999) (width 0.2) (layer B.Cu) (net 2))
+  (segment (start 165.860001 142.439999) (end 166.16 142.14) (width 0.2) (layer B.Cu) (net 2))
+  (segment (start 163.93 143.78) (end 164.52 143.78) (width 0.2) (layer B.Cu) (net 2))
+  (segment (start 166.48 142.14) (end 166.16 142.14) (width 0.2) (layer F.Cu) (net 2))
+  (segment (start 168.175 143.05) (end 167.39 143.05) (width 0.2) (layer F.Cu) (net 2))
+  (segment (start 167.39 143.05) (end 166.48 142.14) (width 0.2) (layer F.Cu) (net 2))
+  (segment (start 169.15 143.05) (end 169.52 142.68) (width 0.2) (layer F.Cu) (net 2))
+  (segment (start 168.175 143.05) (end 169.15 143.05) (width 0.2) (layer F.Cu) (net 2))
+  (segment (start 169.52 142.68) (end 169.52 137.09) (width 0.2) (layer F.Cu) (net 2))
+  (segment (start 168.93 136.5) (end 167.6 136.5) (width 0.2) (layer F.Cu) (net 2))
+  (segment (start 169.52 137.09) (end 168.93 136.5) (width 0.2) (layer F.Cu) (net 2))
+  (segment (start 167.6 136.3) (end 167.6 136.5) (width 0.2) (layer F.Cu) (net 2))
+  (segment (start 167.6 136.5) (end 167.6 137.67) (width 0.2) (layer F.Cu) (net 2))
   (segment (start 168.8 131.4) (end 168.8 131.725) (width 0.2) (layer F.Cu) (net 3))
   (segment (start 168.8 131.43) (end 168.94 131.57) (width 0.2) (layer F.Cu) (net 3))
@@
   (segment (start 168.94 132.710002) (end 168.94 132.710002) (width 0.2) (layer F.Cu) (net 3))
   (segment (start 167.145 128.625) (end 166.7 128.18) (width 0.2) (layer F.Cu) (net 3))
-  (segment (start 166.615 128.18) (end 166.69 128.18) (width 0.2) (layer F.Cu) (net 3))
-  (segment (start 166.075 128.72) (end 166.615 128.18) (width 0.2) (layer F.Cu) (net 3))
-  (segment (start 166.075 129.115) (end 166.075 128.72) (width 0.2) (layer F.Cu) (net 3))
   (segment (start 166.7 128.18) (end 166.69 128.18) (width 0.2) (layer F.Cu) (net 3))
   (segment (start 167.145 129.42) (end 167.145 128.625) (width 0.2) (layer F.Cu) (net 3))
-  (segment (start 168.8 131.075) (end 167.145 129.42) (width 0.2) (layer F.Cu) (net 3))
-  (segment (start 168.8 131.4) (end 168.8 131.075) (width 0.2) (layer F.Cu) (net 3))
   (segment (start 167.145 130.245) (end 167.145 129.42) (width 0.2) (layer F.Cu) (net 3))
   (segment (start 166.01 131.38) (end 167.145 130.245) (width 0.2) (layer F.Cu) (net 3))
@@
   (segment (start 153.024264 105.91) (end 153.34 105.91) (width 0.2) (layer F.Cu) (net 3))
   (via (at 168.94 132.710002) (size 0.6) (drill 0.3) (layers F.Cu B.Cu) (net 3))
-  (segment (start 168.94 137.51) (end 168.94 137.085736) (width 0.2) (layer B.Cu) (net 3))
-  (segment (start 168.94 137.085736) (end 168.94 132.710002) (width 0.2) (layer B.Cu) (net 3))
   (segment (start 168.94 137.51) (end 168.94 137.51) (width 0.2) (layer F.Cu) (net 3))
-  (via (at 168.94 137.51) (size 0.6) (drill 0.3) (layers F.Cu B.Cu) (net 3))
+  (segment (start 166.12 128.18) (end 166.69 128.18) (width 0.2) (layer F.Cu) (net 3))
+  (segment (start 166.075 129.115) (end 166.075 128.225) (width 0.2) (layer F.Cu) (net 3))
+  (segment (start 166.075 128.225) (end 166.12 128.18) (width 0.2) (layer F.Cu) (net 3))
+  (segment (start 167.97 130.245) (end 167.145 130.245) (width 0.2) (layer F.Cu) (net 3))
+  (segment (start 168.8 131.075) (end 167.97 130.245) (width 0.2) (layer F.Cu) (net 3))
+  (segment (start 168.8 131.4) (end 168.8 131.075) (width 0.2) (layer F.Cu) (net 3))
+  (segment (start 168.21 138.21999) (end 168.619991 137.809999) (width 0.2) (layer F.Cu) (net 3))
+  (segment (start 168.619991 137.809999) (end 168.91999 137.51) (width 0.2) (layer F.Cu) (net 3))
+  (segment (start 168.21 140.99) (end 168.21 138.21999) (width 0.2) (layer F.Cu) (net 3))
+  (segment (start 168.94 132.710002) (end 168.94 137.48999) (width 0.2) (layer B.Cu) (net 3))
+  (segment (start 168.94 137.48999) (end 168.91999 137.51) (width 0.2) (layer B.Cu) (net 3))
+  (via (at 168.91999 137.51) (size 0.6) (drill 0.3) (layers F.Cu B.Cu) (net 3))
   (via (at 144.37 136.87) (size 0.8) (drill 0.4) (layers F.Cu B.Cu) (net 4))
   (via (at 146.64 140.08) (size 0.8) (drill 0.4) (layers F.Cu B.Cu) (net 4))
@@
   (segment (start 147.2 109.52) (end 147.2 108.755702) (width 0.2) (layer F.Cu) (net 42))
   (segment (start 150.759865 107.950187) (end 151.184129 107.950187) (width 0.2) (layer F.Cu) (net 42))
+  (segment (start 167.21 144.05) (end 164.764999 141.604999) (width 0.2) (layer F.Cu) (net 42))
+  (segment (start 164.764999 141.604999) (end 164.465 141.305) (width 0.2) (layer F.Cu) (net 42))
+  (segment (start 168.175 144.05) (end 167.21 144.05) (width 0.2) (layer F.Cu) (net 42))
   (via (at 163.92 138.77) (size 0.6) (drill 0.3) (layers F.Cu B.Cu) (net 43))
   (via (at 159.18 137.47) (size 0.6) (drill 0.3) (layers F.Cu B.Cu) (net 43))
@@
   (segment (start 145.759999 107.949999) (end 145.419988 108.29001) (width 0.2) (layer F.Cu) (net 43))
   (segment (start 145.3 110.43) (end 145.3 108.714274) (width 0.2) (layer B.Cu) (net 43))
+  (via (at 166.4 141.29) (size 0.6) (drill 0.3) (layers F.Cu B.Cu) (net 43))
+  (segment (start 168.175 142.05) (end 167.16 142.05) (width 0.2) (layer F.Cu) (net 43))
+  (segment (start 167.16 142.05) (end 166.4 141.29) (width 0.2) (layer F.Cu) (net 43))
+  (segment (start 163.92 138.81) (end 163.92 138.77) (width 0.2) (layer B.Cu) (net 43))
+  (segment (start 166.4 141.29) (end 163.92 138.81) (width 0.2) (layer B.Cu) (net 43))
   (segment (start 143.181974 107.144244) (end 143.181974 106.71998) (width 0.2) (layer B.Cu) (net 44))
   (segment (start 141.49 108.97479) (end 143.181974 107.282816) (width 0.2) (layer B.Cu) (net 44))
@@
   (segment (start 142.736783 106.12893) (end 142.436784 106.428929) (width 0.2) (layer F.Cu) (net 45))
   (segment (start 146.25 105.85) (end 143.015713 105.85) (width 0.2) (layer F.Cu) (net 45))
+  (segment (start 166.169999 138.600001) (end 164.886005 138.600001) (width 0.2) (layer F.Cu) (net 45))
+  (segment (start 166.55 138.22) (end 166.169999 138.600001) (width 0.2) (layer F.Cu) (net 45))
+  (segment (start 166.55 137.245) (end 166.55 138.22) (width 0.2) (layer F.Cu) (net 45))
   (via (at 151.49 90.68) (size 0.6) (drill 0.3) (layers F.Cu B.Cu) (net 49))
   (segment (start 151.789999 90.380001) (end 151.49 90.68) (width 0.2) (layer F.Cu) (net 49))
