File: 月光2/月光2.kicad_pcb (KiCad board)
At the start: 2 copper layers, 40 x 60.5 mm, 69 parts, among them J1 Conn_01x12, J2 Conn_01x12, J3 Conn_01x05, J4 Conn_01x03, J6 Conn_01x02, Q5 IRLML6344TRPBFTR, SW1 SW_Push_Dual_x2, U1 DRV8835, U2 STM32F413CH6, U3 LED_FOTR, U4 LP5907_DBV, U5 ICM20648, U6 LED_FOTR, U7 LED_FOTR, U8 LED_FOTR, Y1 Crystal_GND23

Commit message: finish 5
Routing:
- net encL_2: track 55.0 -> 53.5 mm
- net GND: track 273.3 -> 272.3 mm
- net sens_LL: track 52.5 -> 53.3 mm

Commit message: beta finish
Routing:
- net GND: vias 25 -> 54
- added copper zone on B.Cu, net GND
- added copper zone on F.Cu, net GND
