File: 月光2/_autosave-月光2.kicad_pcb (KiCad board)
At the start: 2 copper layers, 40 x 60.5 mm, 69 parts, among them J1 Conn_01x12, J2 Conn_01x12, J3 Conn_01x05, J4 Conn_01x03, J6 Conn_01x02, Q5 IRLML6344TRPBFTR, SW1 SW_Push_Dual_x2, U1 DRV8835, U2 STM32F413CH6, U3 LED_FOTR, U4 LP5907_DBV, U5 ICM20648, U6 LED_FOTR, U7 LED_FOTR, U8 LED_FOTR, Y1 Crystal_GND23

Commit message: rename
Routing:
- net GND: vias 57 -> 58
Changed lines of the file:
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@@
     (thickness 1.6)
     (drawings 80)
-    (tracks 1305)
+    (tracks 1306)
     (zones 0)
     (modules 69)
@@
   (via (at 152.15 139.33) (size 0.6) (drill 0.3) (layers F.Cu B.Cu) (net 2))
   (via (at 137.46 140.87) (size 0.6) (drill 0.3) (layers F.Cu B.Cu) (net 2))
+  (via (at 157.91 140.27) (size 0.6) (drill 0.3) (layers F.Cu B.Cu) (net 2))
   (segment (start 168.8 131.4) (end 168.8 131.725) (width 0.2) (layer F.Cu) (net 3))
   (segment (start 168.8 131.43) (end 168.94 131.57) (width 0.2) (layer F.Cu) (net 3))
@@
   (segment (start 144.91 98.44) (end 144.91 96.08) (width 0.2) (layer F.Cu) (net 93))
   (segment (start 144.91 96.08) (end 146.23 94.76) (width 0.2) (layer F.Cu) (net 93))
+  (zone (net 2) (net_name GND) (layer B.Cu) (hatch edge 0.508)
+    (connect_pads yes (clearance 0.508))
+    (min_thickness 0.254)
+    (fill yes (arc_segments 32) (thermal_gap 0.508) (thermal_bridge_width 0.508))
+    (polygon
+      (pts
+        (xy 157.14237 104.109571) (xy 157.12 104.13) (xy 157.564199 104.312335) (xy 157.17 104.22) (xy 155.613798 104.342943)
+        (xy 155.332368 103.569012)
+      )
+    )
+  )
   (zone (net 2) (net_name GND) (layer F.Cu) (hatch edge 0.508)
     (connect_pads yes (clearance 0.508))
@@
     (polygon
       (pts
+        (xy 166.89 109.21) (xy 170.78 110.49) (xy 170.9 110.41) (xy 169.59 107.24)
+      )
+    )
+    (polygon
+      (pts
         (xy 140.47 107.87) (xy 140.71 109.45) (xy 143.43 108.93) (xy 143.59 107.76)
       )
@@
     (polygon
       (pts
-        (xy 157.14237 104.109571) (xy 157.12 104.13) (xy 157.564199 104.312335) (xy 157.17 104.22) (xy 155.613798 104.342943)
-        (xy 155.332368 103.569012)
+        (xy 176.58 87.4) (xy 176.58 87.48) (xy 176.56 147.78) (xy 122.42 147.99) (xy 122.43 87.38)
       )
     )
-  )
-  (zone (net 2) (net_name GND) (layer B.Cu) (hatch edge 0.508)
-    (connect_pads yes (clearance 0.508))
-    (min_thickness 0.254)
-    (fill yes (arc_segments 32) (thermal_gap 0.508) (thermal_bridge_width 0.508))
     (polygon
       (pts
-        (xy 176.58 87.4) (xy 176.58 87.48) (xy 176.56 147.78) (xy 122.42 147.99) (xy 122.43 87.38)
+        (xy 138.969197 141.090165) (xy 138.65 141.61) (xy 142.39 141.16) (xy 140.328574 140.194425) (xy 143.2 137.9)
+        (xy 138.94 134.19)
       )
     )
@@
     (polygon
       (pts
-        (xy 155.11 134.18) (xy 160.09 137.12) (xy 162.1 131.06) (xy 157.19 128.86)
+        (xy 160.534602 130.358599) (xy 157.19 128.86) (xy 155.11 134.18) (xy 160.09 137.12) (xy 160.311623 136.451824)
+        (xy 162.45 139.28) (xy 166.77 133.57) (xy 165.809362 133.035869) (xy 161.4 128.51)
       )
     )
@@
       )
     )
+    (polygon
+      (pts
+        (xy 163.27 110.49) (xy 162.75 114.07) (xy 172.28 114.07) (xy 172.78 109.75)
+      )
+    )
