File: gekko/encoder.sch (KiCad schematic (older format))
At the start: 11 parts, among them J1 Conn_01x02_Male, J2 Conn_01x04_Female, J5 Conn_01x02_Male, J7 Conn_01x04_Female, J8 Conn_01x02_Male, J9 Conn_01x02_Male, U10 MA702GQ-P, U11 MA702GQ-P

Commit message: betaGND
Parts:
- removed RN1: R_Pack04_10k, micro:R10k×4, symbol gekko-rescue:R_Pack04-Device
- added R17, R19, R29, R30: 10k, Resistor_SMD:R_0402_1005Metric, symbol Device:R
Connections:
- net +3V3: now also J2.2 (Pin_2), J7.3 (Pin_3); no longer J2.1 (Pin_1), J7.1 (Pin_1)
- net GND: now also J2.1 (Pin_1), J7.4 (Pin_4); no longer C23.2, C24.2, J1.2 (Pin_2), J2.2 (Pin_2), J7.2 (Pin_2), J8.2 (Pin_2), U10.10 (TEST), U10.8 (GND), U11.10 (TEST), U11.8 (GND)
- net encL_1_EXTI_cn: now also R17.1
- net encL_2_EXTI_cn: now also R19.1
- net encR_1_EXTI: now also J7.2 (Pin_2); no longer J7.3 (Pin_3)
- net encR_1_EXTI_cn: now also R29.1
- net encR_2_EXTI: now also J7.1 (Pin_1); no longer J7.4 (Pin_4)
- net encR_2_EXTI_cn: now also R30.1
- net +3.3V renamed +3.3V_L
- net +3.3V_L: now also R17.2, R19.2; no longer C24.1, J8.1 (Pin_1), U11.13 (VDD)
- new net +3.3V_R: C24.1, J8.1 (Pin_1), R29.2, R30.2, U11.13 (VDD)
- new net GND_L: C23.2, J1.2 (Pin_2), U10.10 (TEST), U10.8 (GND)
- new net GND_R: C24.2, J8.2 (Pin_2), U11.10 (TEST), U11.8 (GND)
Other:
- moved on the sheet: C23, C24, J2, J7, U10, U11
