File: gekko/gekko.kicad_pcb (KiCad board)
At the start: 2 copper layers, 40 x 60.5 mm, 70 parts, among them J1 Conn_01x12, J2 Conn_01x12, J3 Conn_01x05, J4 Conn_01x03, J6 Conn_01x02, Q5 IRLML6344TRPBFTR, SW1 SW_Push_Dual_x2, U1 DRV8835, U2 STM32F413CH6, U3 LED_FOTR, U4 LP, U5 ICM20648, U6 LED_FOTR, U7 LED_FOTR, U8 LED_FOTR, Y1 Crystal_GND23

Commit message: PCB
Parts:
- removed D8: 1SMB5928BT3G, micro:PDZ4.3BZ
- removed G***: LOGO, micro:fonto
- added C23: 1μ, Capacitor_SMD:C_0402_1005Metric, F.Cu at (127.5, 138.3)
- added C24: 1μ, Capacitor_SMD:C_0402_1005Metric, F.Cu at (176.5, 142.3)
- added C9: 1μ, Capacitor_SMD:C_0402_1005Metric, F.Cu at (155.2, 140.1)
- added D1: LED_RED, LED_SMD:LED_0402_1005Metric, F.Cu at (128.0, 109.8)
- added D2: LED_RED, LED_SMD:LED_0402_1005Metric, F.Cu at (150.0, 84.3)
- added D3: LED_RED, LED_SMD:LED_0402_1005Metric, F.Cu at (174.0, 99.3)
- added D4: D_TVS, Diode_SMD:D_0402_1005Metric, F.Cu at (164.8, 145.0)
- added J5: Conn_01x02_Male, micro:enc_mount_bk_1, F.Cu at (126.0, 147.8)
- added J7: Conn_01x04_Female, micro:enc_mount_fr_L, F.Cu at (156.4, 119.8)
- added J8: Conn_01x02_Male, micro:enc_mount_bk_1, B.Cu at (170.5, 137.5)
- added J9: Conn_01x02_Male, micro:enc_mount_bk_1, F.Cu at (184.5, 141.3)
- added R11: 330, Resistor_SMD:R_0402_1005Metric, F.Cu at (152.5, 84.3)
- added R12: 330, Resistor_SMD:R_0402_1005Metric, F.Cu at (179.0, 100.3)
- added R13: 10k, Resistor_SMD:R_0402_1005Metric, F.Cu at (160.2, 140.1)
- added R15: 10k, Resistor_SMD:R_0402_1005Metric, F.Cu at (154.4, 134.6)
- added R9: 330, Resistor_SMD:R_0402_1005Metric, F.Cu at (128.0, 106.8)
- added SW2: SW_DPDT_x2, micro:AYZ0102AGRLC, F.Cu at (158.6, 144.5)
- added U10: MA702GQ-P, Package_DFN_QFN:QFN-16-1EP_3x3mm_P0.5mm_EP1.7x1.7mm, F.Cu at (123.6, 137.4)
- added U11: MA702GQ-P, Package_DFN_QFN:QFN-16-1EP_3x3mm_P0.5mm_EP1.7x1.7mm, F.Cu at (176.4, 137.7)
- added U12: sw_pch, micro:SSM3J338R, F.Cu at (160.0, 137.3)
- added U9: RP124N334E-TR-FE, Package_TO_SOT_SMD:SOT-23-5, F.Cu at (156.1, 137.3)
- C1: value 0.1μ -> 1μ
- C19, C20, C21, C22: value 470μ -> 47μ; footprint Capacitor_SMD:C_1812_4532Metric -> Capacitor_SMD:C_0603_1608Metric
- J1: value Conn_01x12 -> Conn_01x02_Male; footprint micro:Molex52745-1297 -> micro:enc_mount_bk_1
- J2: value Conn_01x12 -> Conn_01x04_Female; footprint micro:Molex52745-1297 -> micro:enc_mount_fr_L
- RN1, RN2: value R_Pk4_10k -> R_Pack04_10k
- U4: value LP -> LP5907_DBV
- moved C2 46.0 mm to (120.1, 129.1)
- moved R1 46.0 mm to (120.0, 131.4)
- moved R10 38.1 mm to (121.5, 114.8), turned to 0 degrees
- moved RN1 38.1 mm to (178.0, 148.8), turned to 0 degrees
- moved R14 37.3 mm to (122.0, 119.3)
- moved D5 36.8 mm to (124.5, 114.8)
- moved R18 36.2 mm to (122.0, 122.3)
- moved SW1 35.8 mm to (133.0, 127.8)
- moved D10 35.1 mm to (124.5, 122.3)
- moved J6 35.0 mm to (168.5, 145.8), turned to 90 degrees
- moved D7 34.6 mm to (124.5, 119.3)
- moved J3 34.4 mm to (132.5, 142.3)
- moved J4 34.1 mm to (132.5, 134.8), turned to 90 degrees
- moved C25 33.3 mm to (164.2, 137.1), turned to 0 degrees
- moved U4 33.3 mm to (167.4, 134.9)
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Connections:
- net UART_RX renamed USART_RX
- net UART_TX renamed USART_TX
- C1 pad 1: +3V3 -> GND
- C1 pad 2: GND -> BATT_SW
- C12 pad 1: +3V3 -> battery_wt_vout
- C13 pad 1: +BATT -> BATT_SW
- C14 pad 1: +3V3 -> battery_wt_vout
- C15 pad 1: +3V3 -> battery_wt_vout
- C16 pad 2: +3V3 -> battery_wt_vout
- C18 pad 2: +3V3 -> battery_wt_vout
- C25 pad 1: +BATT -> BATT_SW
- C26 pad 1: +3V3 -> battery_wt_vout
- C3 pad 1: +3V3 -> battery_wt_vout
- C4 pad 2: +BATT -> BATT_SW
- C5 pad 1: +3V3 -> battery_wt
- C7 pad 1: +3V3 -> battery_wt_vout
- C8 pad 1: +3V3 -> battery_wt_vout
- D10 pad 1: LED_3 -> DEBUG_LED3
- D5 pad 1: LED_2 -> DEBUG_LED2
- D7 pad 1: LED_1 -> DEBUG_LED1
- J1 pad 1: MORTOR_1+ -> +3.3V
- J1 pad 2: MORTOR_1- -> GND
- J2 pad 1: MORTOR_2+ -> battery_wt_vout
- J2 pad 2: MORTOR_2- -> GND
- J2 pad 3: Net-(J2-Pad3) -> encL_1_EXTI
- J2 pad 4: GND -> encL_2_EXTI
- J3 pad 1: +3V3 -> battery_wt_vout
- L1 pad 2: +3V3 -> battery_wt_vout
- R1 pad 1: +3V3 -> battery_wt_vout
- R10 pad 1: +3V3 -> battery_wt_vout
- R14 pad 2: +3V3 -> battery_wt_vout
- R16 pad 1: +BATT -> BATT_SW
- R18 pad 2: +3V3 -> battery_wt_vout
- R2 pad 2: RLED_PWM -> R_LED_PWM
- R20 pad 1: +3V3 -> battery_wt_vout
- R26 pad 2: +3V3 -> battery_wt_vout
- R27 pad 2: +3V3 -> battery_wt_vout
- R28 pad 2: +3V3 -> battery_wt_vout
- R4 pad 2: +3V3 -> battery_wt_vout
- RN1 pad 1: encR_1 -> +3.3V
- RN1 pad 2: encR_2 -> +3.3V
- RN1 pad 3: encL_1 -> +3.3V
- RN1 pad 4: encL_2 -> +3.3V
- RN1 pad 5: +3V3 -> encR_2_EXTI_cn
- RN1 pad 6: +3V3 -> encR_1_EXTI_cn
- RN1 pad 7: +3V3 -> encL_2_EXTI_cn
- RN1 pad 8: +3V3 -> encL_1_EXTI_cn
- RN2 pad 5: +3V3 -> battery_wt_vout
- RN2 pad 6: +3V3 -> battery_wt_vout
- RN2 pad 7: +3V3 -> battery_wt_vout
- RN2 pad 8: +3V3 -> battery_wt_vout
- U1 pad 1: +BATT -> BATT_SW
- U1 pad 12: +3V3 -> battery_wt_vout
- U1 pad 2: MORTOR_1+ -> MotorR_Foward
- U1 pad 3: MORTOR_1- -> MotorR_Reverce
- U1 pad 4: MORTOR_2+ -> MotorL_Foward
- U1 pad 5: MORTOR_2- -> MotorL_Reverce
- U2 pad 1: +3V3 -> battery_wt_vout
- U2 pad 10: MotorL_Reverce -> DEBUG_LED3
- U2 pad 11: MotorL_Foward -> MotorL_Reverce
- U2 pad 12: RLED_PWM -> MotorL_Foward
- U2 pad 13: sens_LL -> battery_wt
- U2 pad 17: Net-(U2-Pad17) -> sens_LL
- U2 pad 18: Net-(U2-Pad18) -> R_LED_PWM
- U2 pad 19: LED_3 -> DEBUG_LED4
- U2 pad 20: Net-(U2-Pad20) -> DEBUG_LED5
- U2 pad 21: Net-(U2-Pad21) -> DEBUG_LED6
- U2 pad 32: LED_2 -> Net-(U2-Pad32)
- U2 pad 33: LED_1 -> Net-(U2-Pad33)
- U2 pad 36: +3V3 -> battery_wt_vout
- U2 pad 38: encL_2 -> encL_2_EXTI
- U2 pad 39: encL_1 -> encL_1_EXTI
- U2 pad 4: Net-(U2-Pad4) -> DEBUG_LED1
- U2 pad 40: encR_2 -> encR_2_EXTI
- U2 pad 41: encR_1 -> encR_1_EXTI
- U2 pad 46: Net-(U2-Pad46) -> battery_sw_CE
- U2 pad 48: +3V3 -> battery_wt_vout
- U2 pad 6: Net-(U2-Pad6) -> DEBUG_LED2
- U3 pad 1: +3V3 -> battery_wt_vout
- U4 pad 1: +BATT -> BATT_SW
- U4 pad 3: +BATT -> BATT_SW
- U4 pad 5: +3V3 -> battery_wt_vout
- U5 pad 13: +3V3 -> battery_wt_vout
- U5 pad 8: +3V3 -> battery_wt_vout
- U6 pad 1: +3V3 -> battery_wt_vout
- U7 pad 1: +3V3 -> battery_wt_vout
- U8 pad 1: +3V3 -> battery_wt_vout
- Y1 pad 4: +3V3 -> battery_wt_vout
Routing:
- net GND: track 272.3 -> 0.00 mm, vias 60 -> 0
- net +3V3: track 202.2 -> 0.00 mm, vias 26 -> 0
- net LED_3: track 60.0 -> 0.00 mm, vias 4 -> 0
- net NRST: track 57.2 -> 0.00 mm, vias 4 -> 0
- net USART_TX: track 56.2 -> 0.00 mm, vias 2 -> 0
- net +BATT: track 56.0 -> 0.00 mm, vias 5 -> 0
- net STLINK_TMS: track 55.7 -> 0.00 mm, vias 6 -> 0
- net encL_1: track 55.1 -> 0.00 mm, vias 4 -> 0
- net encL_2: track 53.5 -> 0.00 mm, vias 2 -> 0
- net sens_LL: track 53.3 -> 0.00 mm, vias 4 -> 0
- net USART_RX: track 51.7 -> 0.00 mm, vias 2 -> 0
- net LED_1: track 50.8 -> 0.00 mm, vias 2 -> 0
- net Net-(Q5-Pad2): track 49.2 -> 0.00 mm, vias 6 -> 0
- net STLINK_TCK: track 48.9 -> 0.00 mm, vias 2 -> 0
- net encR_1: track 48.1 -> 0.00 mm, vias 4 -> 0
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- removed copper zone on F.Cu, net GND
Other:
- board size 40 x 60.5 mm -> 58 x 60.5 mm

Commit message: betaGND
Parts:
- removed RN1, RN2: R_Pack04_10k, micro:R10k×4
- added J10: Conn_01x02, micro:motor_pad, F.Cu at (147.2, 132.3)
- added J11: Conn_01x02, micro:motor_pad, F.Cu at (149.5, 136.0)
- added R17: 10k, Resistor_SMD:R_0402_1005Metric, F.Cu at (121.5, 137.3)
- added R19: 10k, Resistor_SMD:R_0402_1005Metric, F.Cu at (123.2, 140.5)
- added R29: 10k, Resistor_SMD:R_0402_1005Metric, F.Cu at (178.5, 136.7)
- added R30: 10k, Resistor_SMD:R_0402_1005Metric, F.Cu at (176.2, 134.5)
- added R31: 10k, Resistor_SMD:R_0402_1005Metric, F.Cu at (152.7, 123.1)
- added R32: 10k, Resistor_SMD:R_0402_1005Metric, F.Cu at (150.2, 115.3)
- added R33: 10k, Resistor_SMD:R_0402_1005Metric, F.Cu at (152.8, 115.3)
- added R34: 10k, Resistor_SMD:R_0402_1005Metric, F.Cu at (147.7, 115.3)
- J5, J9: moved to B.Cu
- J8: moved to F.Cu
- moved R10 39.3 mm to (145.9, 145.5), turned to 270 degrees
- moved D5 38.4 mm to (147.6, 145.5), turned to 270 degrees
- moved C14 36.5 mm to (147.5, 140.5), turned to 270 degrees
- moved C10 35.2 mm to (137.7, 133.0)
- moved C6 33.9 mm to (144.8, 135.0), turned to 315 degrees
- moved Y1 33.6 mm to (146.7, 137.8)
- moved C12 33.5 mm to (133.5, 140.3)
- moved C7 33.5 mm to (145.7, 140.5)
- moved C8 33.5 mm to (144.6, 140.5)
- moved R14 33.3 mm to (142.5, 145.5), turned to 90 degrees
- moved L1 33.1 mm to (146.2, 134.0), turned to 135 degrees
- moved D7 32.9 mm to (144.2, 145.5), turned to 270 degrees
- moved C11 32.0 mm to (135.8, 133.0), turned to 180 degrees
- moved R18 28.9 mm to (139.2, 145.5), turned to 90 degrees
- moved D10 28.5 mm to (140.9, 145.5), turned to 270 degrees
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Connections:
- C23 pad 1: +3.3V -> +3.3V_L
- C23 pad 2: GND -> GND_L
- C24 pad 1: +3.3V -> +3.3V_R
- C24 pad 2: GND -> GND_R
- J1 pad 1: +3.3V -> +3.3V_L
- J1 pad 2: GND -> GND_L
- J2 pad 1: battery_wt_vout -> GND
- J2 pad 2: GND -> battery_wt_vout
- J7 pad 1: battery_wt_vout -> encR_2_EXTI
- J7 pad 2: GND -> encR_1_EXTI
- J7 pad 3: encR_1_EXTI -> battery_wt_vout
- J7 pad 4: encR_2_EXTI -> GND
- J8 pad 1: +3.3V -> +3.3V_R
- J8 pad 2: GND -> GND_R
- SW2 pad 1: Net-(SW2-Pad1) -> GND
- SW2 pad 3: GND -> Net-(SW2-Pad3)
- U1 pad 2: MotorR_Foward -> MotorR_Foward_Out
- U1 pad 3: MotorR_Reverce -> MotorR_Reverce_Out
- U1 pad 4: MotorL_Foward -> MotorL_Foward_Out
- U1 pad 5: MotorL_Reverce -> MotorL_Reverce_Out
- U10 pad 10: GND -> GND_L
- U10 pad 13: +3.3V -> +3.3V_L
- U10 pad 8: GND -> GND_L
- U11 pad 10: GND -> GND_R
- U11 pad 13: +3.3V -> +3.3V_R
- U11 pad 8: GND -> GND_R
- U2 pad 19: DEBUG_LED4 -> DEBUG_LED6
- U2 pad 21: DEBUG_LED6 -> DEBUG_LED4
Routing:
- net battery_wt_vout: track 0.00 -> 302.4 mm, vias 0 -> 14
- net DEBUG_LED5: track 0.00 -> 52.7 mm, vias 0 -> 4
- net sens_RR: track 0.00 -> 50.8 mm, vias 0 -> 1
- net sens_R: track 0.00 -> 48.3 mm, vias 0 -> 2
- net DEBUG_LED6: track 0.00 -> 46.8 mm, vias 0 -> 4
- net Net-(Q5-Pad2): track 0.00 -> 45.8 mm, vias 0 -> 4
- net encR_2_EXTI: track 0.00 -> 39.8 mm, vias 0 -> 2
- net BATT_SW: track 0.00 -> 39.2 mm
- net GND: track 0.00 -> 39.1 mm, vias 0 -> 1
- net NRST: track 0.00 -> 37.2 mm, vias 0 -> 4
- net sens_L: track 0.00 -> 37.1 mm, vias 0 -> 2
- net encR_1_EXTI: track 0.00 -> 36.1 mm, vias 0 -> 2
- net MOSI_IMU: track 0.00 -> 34.4 mm, vias 0 -> 2
- net SCK_IMU: track 0.00 -> 33.5 mm, vias 0 -> 3
- net encL_1_EXTI: track 0.00 -> 32.9 mm, vias 0 -> 2
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- added copper zone on F.Cu, net (none)
- removed copper zone on B.Cu, net GND
Other:
- rule via_min_drill: 0.3 -> 0.1
- rule via_min_size: 0.4 -> 0.2

Commit message: betaGND
Parts:
- moved J4 1.00 mm to (133.0, 129.8)
- moved D10 0.71 mm to (141.4, 146.0)
- moved D5 0.71 mm to (148.1, 146.0)
- moved D7 0.71 mm to (144.7, 146.0)
- moved R10 0.71 mm to (146.4, 146.0)
- moved R14 0.71 mm to (143.0, 146.0)
- moved R18 0.71 mm to (139.7, 146.0)
Routing:
- net battery_wt_vout: track 302.4 -> 322.7 mm, vias 14 -> 15
- net GND: track 39.1 -> 48.7 mm, vias 1 -> 8
- net Net-(R13-Pad2): track 2.72 -> 5.86 mm, vias 2 -> 3
- net NRST: track 37.2 -> 38.6 mm
- net Net-(Q5-Pad2): track 45.8 -> 47.2 mm, vias 4 -> 3
- net USART_RX: track 8.10 -> 9.04 mm
- net USART_TX: track 7.11 -> 8.04 mm
- net DEBUG_LED3: track 13.5 -> 14.2 mm
- net MISO_IMU: track 31.8 -> 32.3 mm
- added copper zone on F.Cu, net GND
- removed copper zone on F.Cu, net (none)

Commit message: betaGND_B
Routing:
- net GND: track 48.7 -> 138.2 mm, vias 8 -> 22
- net DEBUG_LED3: track 14.2 -> 12.9 mm, vias 4 -> 2
- net DEBUG_LED2: track 17.9 -> 18.8 mm
- net battery_wt_vout: track 322.7 -> 322.6 mm, vias 15 -> 17
- added copper zone on B.Cu, net GND

Commit message: finish
Parts:
- added G***: LOGO, micro:fonto, B.Cu at (145.0, 145.0)
- moved C24 1.50 mm to (177.3, 140.5)
- moved R30 1.00 mm to (177.2, 134.5)
- moved R29 1.00 mm to (179.5, 136.7)
- moved C23 1.00 mm to (123.2, 134.5)
- moved R19 1.00 mm to (122.2, 140.5)
- moved R17 1.00 mm to (120.5, 137.3)
- moved J8 0.80 mm to (171.2, 137.5)
- moved J9 0.80 mm to (171.2, 137.5)
- moved J1 0.80 mm to (128.8, 137.5)
- moved J5 0.80 mm to (128.8, 137.5)
- moved U11 0.70 mm to (176.2, 137.5)
- moved U10 0.70 mm to (123.8, 137.5)
Routing:
- net GND: track 138.2 -> 145.2 mm, vias 22 -> 111
- net GND_R: track 12.5 -> 14.8 mm
- net GND_L: track 16.4 -> 14.3 mm
- net +3.3V_L: track 13.9 -> 15.9 mm
- net +3.3V_R: track 16.0 -> 17.2 mm
- net SCK_IMU: track 33.4 -> 32.5 mm
- net encL_1_EXTI_cn: track 11.3 -> 12.1 mm
- net encL_2_EXTI_cn: track 9.77 -> 10.6 mm
- net encR_1_EXTI_cn: track 8.93 -> 9.59 mm
Other:
- board size 58 x 60.5 mm -> 60 x 60.5 mm

Commit message: RE_patern
Parts:
- removed C13, C15: 22μ, micro:6SVP22M
- removed G***: LOGO, micro:fonto
- removed Q5: IRLML6344TRPBFTR, micro:IRFML8244TRPBF
- added Q1: Q_NMOS_GSD, Package_TO_SOT_SMD:SOT-23, F.Cu at (139.8, 107.2)
- R16: value 140 -> 165
- moved C9 12.7 mm to (163.8, 130.0), turned to 90 degrees
- moved C5 12.6 mm to (163.8, 128.0), turned to 90 degrees
- moved U9 12.1 mm to (166.5, 129.5)
- moved SW1 11.2 mm to (135.5, 146.0), turned to 180 degrees
- moved R15 11.2 mm to (169.0, 129.0), turned to 90 degrees
- moved J10 11.0 mm to (158.2, 133.6), turned to 135 degrees
- moved C1 10.8 mm to (168.5, 132.5), turned to 0 degrees
- moved C2 8.70 mm to (137.2, 145.5), turned to 90 degrees
- moved J3 6.29 mm to (132.6, 139.0), turned to 90 degrees
- moved U12 5.71 mm to (165.0, 141.0)
- moved C14 5.59 mm to (152.5, 138.0), turned to 0 degrees
- moved R13 5.24 mm to (162.5, 140.5), turned to 135 degrees
- moved J11 5.23 mm to (154.2, 133.8), turned to 225 degrees
- moved R1 5.00 mm to (131.2, 145.5), turned to 270 degrees
- moved C12 4.60 mm to (137.8, 142.0), turned to 180 degrees
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Routing:
- net GND: track 145.6 -> 34.9 mm, vias 111 -> 29
- net battery_wt_vout: track 322.4 -> 272.8 mm, vias 17 -> 5
- net encR_2_EXTI: track 39.9 -> 0.00 mm, vias 2 -> 0
- net encR_1_EXTI: track 36.6 -> 0.00 mm, vias 2 -> 0
- net MOSI_IMU: track 34.1 -> 0.00 mm, vias 2 -> 0
- net encL_1_EXTI: track 33.4 -> 0.00 mm, vias 2 -> 0
- net SCK_IMU: track 32.5 -> 0.32 mm, vias 3 -> 0
- net MISO_IMU: track 32.3 -> 0.36 mm, vias 2 -> 0
- net CS_IMU: track 30.1 -> 0.00 mm
- net encL_2_EXTI: track 29.1 -> 0.00 mm, vias 2 -> 0
- net DEBUG_LED6: track 46.8 -> 23.2 mm, vias 4 -> 2
- net MotorL_Foward: track 20.6 -> 9.41 mm
- net sens_RR: track 50.8 -> 40.3 mm, vias 1 -> 0
- net MotorL_Reverce: track 20.8 -> 10.6 mm
- net DEBUG_LED2: track 18.8 -> 8.68 mm
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- removed copper zone on B.Cu, net GND

Commit message: RE_patern_finish
Parts:
- moved R34 9.62 mm to (153.3, 123.2)
- moved R33 8.84 mm to (148.8, 123.2)
- moved C18 8.05 mm to (153.8, 121.2)
- moved R32 7.88 mm to (146.8, 122.4), turned to 270 degrees
- moved C17 7.54 mm to (153.8, 119.0), turned to 270 degrees
- moved R31 7.44 mm to (146.2, 119.8)
- moved C16 7.03 mm to (150.5, 116.3)
- moved J4 0.36 mm to (132.6, 131.1)
- moved R13 0.27 mm to (162.4, 140.8), turned to 90 degrees
- turned U5 to 90 degrees
Routing:
- net encR_2_EXTI: track 0.00 -> 39.8 mm, vias 0 -> 2
- net encR_1_EXTI: track 0.00 -> 36.6 mm, vias 0 -> 2
- net encL_1_EXTI: track 0.00 -> 32.9 mm, vias 0 -> 2
- net battery_wt_vout: track 272.8 -> 304.1 mm, vias 5 -> 8
- net encL_2_EXTI: track 0.00 -> 28.0 mm, vias 0 -> 2
- net MISO_IMU: track 0.36 -> 24.8 mm, vias 0 -> 2
- net DEBUG_LED6: track 23.2 -> 45.4 mm
- net MOSI_IMU: track 0.00 -> 20.7 mm, vias 0 -> 2
- net SCK_IMU: track 0.32 -> 20.6 mm, vias 0 -> 2
- net CS_IMU: track 0.00 -> 20.3 mm, vias 0 -> 2
- net sens_RR: track 40.3 -> 46.7 mm, vias 0 -> 1
- net sens_R: track 38.6 -> 44.5 mm, vias 1 -> 2
- net MotorR_Foward_Out: track 3.07 -> 4.30 mm
- net MotorL_Foward_Out: track 3.28 -> 4.37 mm
- net MotorL_Reverce_Out: track 2.72 -> 3.36 mm
