File: gekko/gekko.kicad_pcb (KiCad board)
At the start: 2 copper layers, 60 x 60.5 mm, 95 parts, among them J1 Conn_01x02_Male, J10 Conn_01x02, J11 Conn_01x02, J2 Conn_01x04_Female, J3 Conn_01x05, J4 Conn_01x03, J5 Conn_01x02_Male, J6 Conn_01x02, J7 Conn_01x04_Female, J8 Conn_01x02_Male, J9 Conn_01x02_Male, Q1 Q_NMOS_GSD, SW1 SW_Push_Dual_x2, SW2 SW_DPDT_x2, U1 DRV8835, U10 MA702GQ-P, U11 MA702GQ-P, U12 sw_pch, U2 STM32F413CH6, U3 LED_FOTR, U4 LP5907_DBV, U5 ICM20648, U6 LED_FOTR, U7 LED_FOTR, U8 LED_FOTR, U9 RP124N334E-TR-FE, Y1 Crystal_GND23

Commit message: RE_patern_finish_2
Parts:
- moved D6 2.50 mm to (161.5, 133.0)
- moved R16 2.50 mm to (161.5, 134.2), turned to 180 degrees
- moved D9 2.36 mm to (163.8, 133.0), turned to 0 degrees
- moved R20 2.36 mm to (163.8, 134.2)
- moved C4 1.04 mm to (159.7, 136.5), turned to 90 degrees
- moved C25 0.98 mm to (166.6, 138.7), turned to 0 degrees
Routing:
- net GND: track 34.9 -> 53.4 mm, vias 29 -> 1
- net BATT_SW: track 31.3 -> 32.9 mm
- net battery_wt_vout: track 304.1 -> 305.1 mm
- net Net-(Q1-Pad3): track 46.9 -> 46.0 mm, vias 3 -> 2

Commit message: RE_beta_finish
Routing:
- net GND: track 53.4 -> 95.4 mm, vias 1 -> 68
- net encL_2_EXTI: track 28.0 -> 26.8 mm
- net encL_1_EXTI: track 32.9 -> 31.8 mm
- net encR_2_EXTI: track 39.8 -> 38.8 mm
- net DEBUG_LED2: track 8.68 -> 9.46 mm
- net encR_1_EXTI: track 36.6 -> 35.9 mm
- added copper zone on B.Cu, net GND

Commit message: For the time being
Parts:
- added G***: LOGO, micro:fonto, B.Cu at (145.3, 145.0)
Routing:
- net GND: vias 68 -> 69
