File: gekko/gekko.sch (KiCad schematic (older format))
At the start: 69 parts, among them J1 Conn_01x12, J2 Conn_01x12, J3 Conn_01x05, J4 Conn_01x03, J6 Conn_01x02, Q5 IRLML6344TRPBFTR, SW1 SW_Push_Dual_x2, U1 DRV8835, U2 STM32F413CH6, U3 LED_FOTR, U4 LP5907_DBV, U5 ICM20648, U6 LED_FOTR, U7 LED_FOTR, U8 LED_FOTR, Y1 Crystal_GND23

Commit message: new_re
Parts:
- C1, C10, C11, C12, C14, C16, C17, C18, C19, C2, C20, C21, C22, C25, C26, C3, C4, C5, C6, C7, C8: symbol Device:C -> gekko-rescue:C-Device
- C13, C15: symbol Device:CP -> gekko-rescue:CP-Device
- D10, D5, D6, D7, D9: symbol Device:LED -> gekko-rescue:LED-Device
- D8: symbol Device:D -> gekko-rescue:D-Device
- J1, J2: symbol Connector_Generic:Conn_01x12 -> gekko-rescue:Conn_01x12-Connector_Generic
- J3: symbol Connector_Generic:Conn_01x05 -> gekko-rescue:Conn_01x05-Connector_Generic
- J4: symbol Connector_Generic:Conn_01x03 -> gekko-rescue:Conn_01x03-Connector_Generic
- J6: symbol Connector_Generic:Conn_01x02 -> gekko-rescue:Conn_01x02-Connector_Generic
- L1: symbol Device:L -> gekko-rescue:L-Device
- Q5: symbol Device:Q_NMOS_GDS -> gekko-rescue:Q_NMOS_GDS-Device
- R1, R10, R14, R16, R18, R2, R20, R21, R22, R23, R24, R25, R26, R27, R28, R3, R4, R5, R6, R7, R8: symbol Device:R -> gekko-rescue:R-Device
- RN1, RN2: symbol Device:R_Pack04 -> gekko-rescue:R_Pack04-Device
- U1: symbol mausu:DRV8835 -> gekko-rescue:DRV8835-mausu
- U2: symbol mausu:STM32F413CH6 -> gekko-rescue:STM32F413CH6-mausu
- U3, U6, U7, U8: symbol mausu:LED_FOTR -> gekko-rescue:LED_FOTR-mausu
- U4: symbol mausu:LP5907_DBV -> gekko-rescue:LP5907_DBV-mausu
- U5: symbol mausu:ICM20648 -> gekko-rescue:ICM20648-mausu
- Y1: symbol Device:Crystal_GND23 -> gekko-rescue:Crystal_GND23-Device
Connections:
- net labels added: DEBUG_LED1, DEBUG_LED2, DEBUG_LED3, DEBUG_LED4, DEBUG_LED5, DEBUG_LED6, R_LED_PWM, USART_RX, USART_TX, battery_watch, encL_1_EXTI, encL_2_EXTI, encR_1_EXTI, encR_2_EXTI
- no-connect marks 39 -> 35

Commit message: PCB
Parts:
- removed C1, C5: 0.1μ, Capacitor_SMD:C_0402_1005Metric, symbol gekko-rescue:C-Device
- removed D8: 1SMB5928BT3G, micro:PDZ4.3BZ, symbol gekko-rescue:D-Device
- removed J1, J2: Conn_01x12, micro:Molex52745-1297, symbol gekko-rescue:Conn_01x12-Connector_Generic
- removed RN1: R_Pack04_10k, micro:R10k×4, symbol gekko-rescue:R_Pack04-Device
- added C1, C9: 1μ, Capacitor_SMD:C_0402_1005Metric, symbol Device:C
- added C5: 0.1μ, Capacitor_SMD:C_0402_1005Metric, symbol Device:C
- added D1, D2, D3: LED_RED, LED_SMD:LED_0402_1005Metric, symbol gekko-rescue:LED-Device
- added D4: D_TVS, Diode_SMD:D_0402_1005Metric, symbol Device:D_TVS
- added R11, R12, R9: 330, Resistor_SMD:R_0402_1005Metric, symbol gekko-rescue:R-Device
- added R13, R15: 10k, Resistor_SMD:R_0402_1005Metric, symbol Device:R
- added SW2: SW_DPDT_x2, micro:AYZ0102AGRLC, symbol Switch:SW_DPDT_x2
- added U12: sw_pch, micro:SSM3J338R, symbol gekko-rescue:sw_pch
- added U9: RP124N334E-TR-FE, Package_TO_SOT_SMD:SOT-23-5, symbol gekko-rescue:RP124N334E-TR-FE
- C19, C20, C21, C22: value 470μ -> 47μ; footprint Capacitor_SMD:C_1812_4532Metric -> Capacitor_SMD:C_0603_1608Metric
Connections:
- net LED_1 is gone; now on net DEBUG_LED1: D7.1 (K)
- net LED_2 is gone; now on net DEBUG_LED2: D5.1 (K)
- net LED_3 is gone; now on net DEBUG_LED3: D10.1 (K)
- net MORTOR_1+ is gone; now on net MotorR_Foward: U1.2 (AOUT1)
- net MORTOR_1- is gone; now on net MotorR_Reverce: U1.3 (AOUT2)
- net MORTOR_2+ is gone; now on net MotorL_Foward: U1.4 (BOUT1)
- net MORTOR_2- is gone; now on net MotorL_Reverce: U1.5 (BOUT2)
- net RLED_PWM is gone; now on net R_LED_PWM: R2.2
- net UART_RX is gone; now on net USART_RX: J4.1 (Pin_1)
- net UART_TX is gone; now on net USART_TX: J4.2 (Pin_2)
- net +3V3: now also C9.1, R11.1, R12.2, R9.2, U9.5 (VOUT)
- net +BATT: now also D4.1 (A1), R13.1, U12.2 (S); no longer C13.1, C25.1, C4.2, R16.1, U1.1 (VM), U4.1 (IN), U4.3 (EN)
- net DEBUG_LED4: now also D1.1 (K)
- net DEBUG_LED5: now also D2.1 (K)
- net DEBUG_LED6: now also D3.1 (K)
- net GND: now also C1.1, C5.2, C9.2, D4.2 (A2), R15.1, SW2.3 (C), U9.2 (GND)
- net battery_sw_CE: now reaches U2.46 (PB9)
- net battery_sw_CE: now also R15.2, U9.3 (CE)
- net battery_watch renamed battery_wt
- net battery_wt: now also C5.1, U9.4 (BN)
- new net: D3.2 (A), R12.1
- new net: D2.2 (A), R11.2
- new net: D1.2 (A), R9.1
- new net: R13.2, SW2.2 (B), U12.1 (G)
- new net BATT_SW: C1.2, C13.1, C25.1, C4.2, R16.1, U1.1 (VM), U12.3 (D), U4.1 (IN), U4.3 (EN), U9.1 (VDD)
- no-connect marks 35 -> 23
Other:
- note added: "BATTERY_WATCH\n\n"
- note added: "FET_SW\n"
- moved on the sheet: C12, C13, C15, C16, C2, C25, C26, D10, D5, D6, D7, D9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

Commit message: betaGND
Parts:
- removed RN2: R_Pack04_10k, micro:R10k×4, symbol gekko-rescue:R_Pack04-Device
- added J10, J11: Conn_01x02, micro:motor_pad, symbol Connector_Generic:Conn_01x02
- added R31, R32, R33, R34: 10k, Resistor_SMD:R_0402_1005Metric, symbol Device:R
Connections:
- net +3V3: now also R31.1, R32.1, R33.1, R34.1
- net CS_IMU: now also R31.2
- net DEBUG_LED4: now also U2.21 (PB10); no longer U2.19 (PB1)
- net DEBUG_LED6: now also U2.19 (PB1); no longer U2.21 (PB10)
- net MISO_IMU: now also R34.2
- net MOSI_IMU: now also R33.2
- net MotorL_Foward: no longer U1.4 (BOUT1)
- net MotorL_Reverce: no longer U1.5 (BOUT2)
- net MotorR_Foward: no longer U1.2 (AOUT1)
- net MotorR_Reverce: no longer U1.3 (AOUT2)
- net SCK_IMU: now also R32.2
- new net MotorL_Foward_Out: J11.1 (Pin_1), U1.4 (BOUT1)
- new net MotorL_Reverce_Out: J11.2 (Pin_2), U1.5 (BOUT2)
- new net MotorR_Foward_Out: J10.1 (Pin_1), U1.2 (AOUT1)
- new net MotorR_Reverce_Out: J10.2 (Pin_2), U1.3 (AOUT2)
Changed lines of the file:
@@
 	7700 1350 7850 1350
-Wire Wire Line
-	7850 5050 7950 5050
-Connection ~ 7950 5050
-Wire Wire Line
-	7950 5050 8050 5050
-Connection ~ 8050 5050
-Wire Wire Line
-	8050 5050 8150 5050
-Connection ~ 8150 5050
-Wire Wire Line
-	8150 5050 9600 5050
 Wire Wire Line
 	2400 1900 2400 2250
@@
 	1150 2550 1600 2550
 Connection ~ 1600 2550
-Wire Wire Line
-	7850 5050 7850 5350
-Wire Wire Line
-	7950 5050 7950 5350
-Wire Wire Line
-	8050 5050 8050 5350
-Wire Wire Line
-	8150 5050 8150 5350
 Connection ~ 1300 5800
 Connection ~ 3650 5800
@@
 $EndComp
 Text GLabel 2450 1600 2    50   Input ~ 0
-MotorR_Foward
+MotorR_Foward_Out
 Text GLabel 2450 1750 2    50   Input ~ 0
-MotorR_Reverce
+MotorR_Reverce_Out
 Text GLabel 2450 2250 2    50   Input ~ 0
-MotorL_Foward
+MotorL_Foward_Out
 Text GLabel 2450 2400 2    50   Input ~ 0
-MotorL_Reverce
+MotorL_Reverce_Out
 Wire Wire Line
 	9300 1100 9450 1100
@@
 Wire Wire Line
 	8000 1700 8000 2050
-$Comp
-L gekko-rescue:R_Pack04-Device RN2
-U 1 1 5DCEEB11
-P 8050 5550
-F 0 "RN2" H 8238 5596 50  0000 L CNN
-F 1 "R_Pack04_10k" H 8238 5505 50  0000 L CNN
-F 2 "micro:R10k×4" V 8325 5550 50  0001 C CNN
-F 3 "~" H 8050 5550 50  0001 C CNN
-	1    8050 5550
-	1    0    0    -1
-$EndComp
 Wire Wire Line
 	7600 5800 7850 5800
-Wire Wire Line
-	7600 5900 7950 5900
-Wire Wire Line
-	7600 6000 8050 6000
-Wire Wire Line
-	7600 6350 8150 6350
-Wire Wire Line
-	7850 5750 7850 5800
 Connection ~ 7850 5800
 Wire Wire Line
 	7850 5800 8800 5800
-Wire Wire Line
-	7950 5750 7950 5900
-Connection ~ 7950 5900
-Wire Wire Line
-	7950 5900 8800 5900
-Wire Wire Line
-	8050 5750 8050 6000
-Connection ~ 8050 6000
-Wire Wire Line
-	8050 6000 8800 6000
-Wire Wire Line
-	8150 5750 8150 6350
-Connection ~ 8150 6350
-Wire Wire Line
-	8150 6350 9950 6350
 Wire Wire Line
 	9300 4250 10050 4250
@@
 Text GLabel 6000 5100 3    50   Input ~ 0
 R_LED_PWM
-Text GLabel 6100 5100 3    50   Input ~ 0
+Text GLabel 6300 5100 3    50   Input ~ 0
 DEBUG_LED4
 Text GLabel 6200 5100 3    50   Input ~ 0
 DEBUG_LED5
-Text GLabel 6300 5100 3    50   Input ~ 0
+Text GLabel 6100 5100 3    50   Input ~ 0
 DEBUG_LED6
 Text GLabel 5050 3900 0    50   Input ~ 0
@@
 $EndComp
 Connection ~ 6750 1500
+$Comp
+L Connector_Generic:Conn_01x02 J10
+U 1 1 5E8A933C
+P 1550 2900
+F 0 "J10" H 1630 2892 50  0000 L CNN
+F 1 "Conn_01x02" H 1630 2801 50  0000 L CNN
+F 2 "micro:motor_pad" H 1550 2900 50  0001 C CNN
+F 3 "~" H 1550 2900 50  0001 C CNN
+	1    1550 2900
+	1    0    0    -1
+$EndComp
+$Comp
+L Connector_Generic:Conn_01x02 J11
+U 1 1 5E8A9ADA
+P 1550 3200
+F 0 "J11" H 1630 3192 50  0000 L CNN
+F 1 "Conn_01x02" H 1630 3101 50  0000 L CNN
+F 2 "micro:motor_pad" H 1550 3200 50  0001 C CNN
+F 3 "~" H 1550 3200 50  0001 C CNN
+	1    1550 3200
+	1    0    0    -1
+$EndComp
+Text GLabel 1350 2900 0    50   Input ~ 0
+MotorR_Foward_Out
+Text GLabel 1350 3000 0    50   Input ~ 0
+MotorR_Reverce_Out
+Text GLabel 1350 3200 0    50   Input ~ 0
+MotorL_Foward_Out
+Text GLabel 1350 3300 0    50   Input ~ 0
+MotorL_Reverce_Out
+$Comp
+L Device:R R?
+U 1 1 5E8AD0AA
+P 7850 5550
+AR Path="/5E9237A4/5E8AD0AA" Ref="R?"  Part="1"
+AR Path="/5E8AD0AA" Ref="R31"  Part="1"
+F 0 "R31" H 7700 5700 50  0000 L CNN
+F 1 "10k" H 7700 5400 50  0000 L CNN
+F 2 "Resistor_SMD:R_0402_1005Metric" V 7780 5550 50  0001 C CNN
+F 3 "~" H 7850 5550 50  0001 C CNN
+	1    7850 5550
+	1    0    0    -1
+$EndComp
+$Comp
+L Device:R R?
+U 1 1 5E8AD0B0
+P 8150 5550
+AR Path="/5E9237A4/5E8AD0B0" Ref="R?"  Part="1"
+AR Path="/5E8AD0B0" Ref="R33"  Part="1"
+F 0 "R33" H 8000 5700 50  0000 L CNN
+F 1 "10k" H 8000 5400 50  0000 L CNN
+F 2 "Resistor_SMD:R_0402_1005Metric" V 8080 5550 50  0001 C CNN
+F 3 "~" H 8150 5550 50  0001 C CNN
+	1    8150 5550
+	1    0    0    -1
+$EndComp
+$Comp
+L Device:R R?
+U 1 1 5E8C01C2
+P 8000 5550
+AR Path="/5E9237A4/5E8C01C2" Ref="R?"  Part="1"
+AR Path="/5E8C01C2" Ref="R32"  Part="1"
+F 0 "R32" H 7850 5700 50  0000 L CNN
+F 1 "10k" H 7850 5400 50  0000 L CNN
+F 2 "Resistor_SMD:R_0402_1005Metric" V 7930 5550 50  0001 C CNN
+F 3 "~" H 8000 5550 50  0001 C CNN
+	1    8000 5550
+	1    0    0    -1
+$EndComp
+$Comp
+L Device:R R?
+U 1 1 5E8C01C8
+P 8300 5550
+AR Path="/5E9237A4/5E8C01C8" Ref="R?"  Part="1"
+AR Path="/5E8C01C8" Ref="R34"  Part="1"
+F 0 "R34" H 8150 5700 50  0000 L CNN
+F 1 "10k" H 8150 5400 50  0000 L CNN
+F 2 "Resistor_SMD:R_0402_1005Metric" V 8230 5550 50  0001 C CNN
+F 3 "~" H 8300 5550 50  0001 C CNN
+	1    8300 5550
+	1    0    0    -1
+$EndComp
+Connection ~ 8000 5050
+Wire Wire Line
+	7850 5050 8000 5050
+Connection ~ 8150 5050
+Wire Wire Line
+	8000 5050 8150 5050
+Connection ~ 8300 5050
+Wire Wire Line
+	8300 5050 9600 5050
+Wire Wire Line
+	8150 5050 8300 5050
+Connection ~ 8000 5900
+Wire Wire Line
+	8000 5900 8800 5900
+Wire Wire Line
+	7600 5900 8000 5900
+Connection ~ 8150 6000
+Wire Wire Line
+	8150 6000 8800 6000
+Wire Wire Line
+	7600 6000 8150 6000
+Connection ~ 8300 6350
+Wire Wire Line
+	8300 6350 9950 6350
+Wire Wire Line
+	7600 6350 8300 6350
+Wire Wire Line
+	7850 5700 7850 5800
+Wire Wire Line
+	8000 5700 8000 5900
+Wire Wire Line
+	8150 5700 8150 6000
+Wire Wire Line
+	8300 5700 8300 6350
+Wire Wire Line
+	7850 5050 7850 5400
+Wire Wire Line
+	8000 5050 8000 5400
+Wire Wire Line
+	8150 5050 8150 5400
+Wire Wire Line
+	8300 5050 8300 5400
 $EndSCHEMATC

Commit message: betaGND
Connections:
- net GND: now also SW2.1 (A); no longer SW2.3 (C)
Changed lines of the file:
@@
 L power:GND #PWR021
 U 1 1 5EA1CF16
-P 6650 2000
-F 0 "#PWR021" H 6650 1750 50  0001 C CNN
-F 1 "GND" H 6655 1827 50  0000 C CNN
-F 2 "" H 6650 2000 50  0001 C CNN
-F 3 "" H 6650 2000 50  0001 C CNN
-	1    6650 2000
+P 6850 2000
+F 0 "#PWR021" H 6850 1750 50  0001 C CNN
+F 1 "GND" H 6855 1827 50  0000 C CNN
+F 2 "" H 6850 2000 50  0001 C CNN
+F 3 "" H 6850 2000 50  0001 C CNN
+	1    6850 2000
 	1    0    0    -1
 $EndComp
@@
 Wire Wire Line
 	4800 7100 4800 7200
-NoConn ~ 6850 2000
+NoConn ~ 6650 2000
 Text GLabel 5800 1150 0    50   Input ~ 0
 USART_RX

Commit message: hattyu_v2
Parts:
- removed C13, C15: 22μ, micro:6SVP22M, symbol gekko-rescue:CP-Device
- R16: value 140 -> 165
- U1: manf# (none) -> 296-30391-1-ND
- U2: manf# (none) -> 497-17018-ND
- U4: manf# (none) -> 296-38557-1-ND
- U5: manf# (none) -> 1428-1061-1-ND
- Y1: manf# (none) -> 535-11177-1-ND
Connections:
- net GND: now also Q5.2 (D); no longer Q5.3 (S)
- net at U3.4 (K), U6.4 (K), U7.4 (K)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: now also Q5.3 (S); no longer Q5.2 (D)
Other:
- note added: "gate_R\n\n"
Changed lines of the file:
@@
 F 3 "~" H 5850 7250 50  0001 C CNN
 	1    5850 7250
-	-1   0    0    -1
+	-1   0    0    1
 $EndComp
 Wire Wire Line
@@
 	7850 1100 7850 1350
 $Comp
-L gekko-rescue:CP-Device C13
-U 1 1 5E705C44
-P 9450 1550
-F 0 "C13" H 9500 1650 50  0000 L CNN
-F 1 "22μ" H 9500 1450 50  0000 L CNN
-F 2 "micro:6SVP22M" H 9488 1400 50  0001 C CNN
-F 3 "~" H 9450 1550 50  0001 C CNN
-	1    9450 1550
-	1    0    0    -1
-$EndComp
-Wire Wire Line
-	9450 1100 9450 1400
-Wire Wire Line
-	9450 2050 9450 1700
-$Comp
 L gekko-rescue:R-Device R16
 U 1 1 5E72594D
 P 8850 1350
 F 0 "R16" H 8920 1396 50  0000 L CNN
-F 1 "140" H 8920 1305 50  0000 L CNN
+F 1 "165" H 8920 1305 50  0000 L CNN
 F 2 "Resistor_SMD:R_0402_1005Metric" V 8780 1350 50  0001 C CNN
 F 3 "~" H 8850 1350 50  0001 C CNN
@@
 F 2 "micro:DRV8835DSSR" H 1700 1100 50  0001 C CNN
 F 3 "" H 1700 1100 50  0001 C CNN
+F 4 "296-30391-1-ND" H 1700 1450 50  0001 C CNN "manf#"
 	1    1700 1450
 	1    0    0    -1
@@
 F 2 "micro:STM32F411CEU6" H 6050 3200 50  0001 C CNN
 F 3 "" H 6050 3200 50  0001 C CNN
+F 4 "497-17018-ND" H 6050 3200 50  0001 C CNN "manf#"
 	1    6050 3200
 	1    0    0    -1
@@
 F 2 "micro:ICM20648" H 9350 3900 50  0001 C CNN
 F 3 "" H 9350 3900 50  0001 C CNN
+F 4 "1428-1061-1-ND" H 9350 5200 50  0001 C CNN "manf#"
 	1    9350 5200
 	1    0    0    -1
@@
 F 2 "micro:LP5907MFX-3.3&slash_NOPB" H 10100 1000 50  0001 C CNN
 F 3 "" H 10100 1000 50  0001 C CNN
+F 4 "296-38557-1-ND" H 10100 1000 50  0001 C CNN "manf#"
 	1    10100 1000
 	1    0    0    -1
@@
 NoConn ~ 10350 1300
 $Comp
-L gekko-rescue:CP-Device C15
-U 1 1 5DA4AB68
-P 10600 1550
-F 0 "C15" H 10718 1596 50  0000 L CNN
-F 1 "22μ" H 10718 1505 50  0000 L CNN
-F 2 "micro:6SVP22M" H 10638 1400 50  0001 C CNN
-F 3 "~" H 10600 1550 50  0001 C CNN
-	1    10600 1550
-	1    0    0    -1
-$EndComp
-Wire Wire Line
-	10600 1100 10600 1400
-Wire Wire Line
-	10600 1700 10600 2050
-$Comp
 L gekko-rescue:Crystal_GND23-Device Y1
 U 1 1 5DA8662B
@@
 F 2 "micro:crystal" H 10200 4500 50  0001 C CNN
 F 3 "~" H 10200 4500 50  0001 C CNN
+F 4 "535-11177-1-ND" H 10200 4500 50  0001 C CNN "manf#"
 	1    10200 4500
 	-1   0    0    -1
@@
 Wire Wire Line
 	10850 1950 10850 2050
-Wire Wire Line
-	10850 2050 10600 2050
 Text Notes 8450 4900 0    157  ~ 0
 IMU
@@
 Wire Wire Line
 	9700 1700 9700 2050
-Connection ~ 10600 1100
-Wire Wire Line
-	10600 1100 10750 1100
-Connection ~ 10600 2050
 Wire Wire Line
 	9800 2050 10400 2050
@@
 Connection ~ 10400 1100
 Wire Wire Line
-	10400 1100 10600 1100
-Wire Wire Line
 	10400 1700 10400 2050
 Connection ~ 10400 2050
-Wire Wire Line
-	10400 2050 10600 2050
 Wire Wire Line
 	6100 7250 6100 7500
@@
 Text GLabel 2450 2400 2    50   Input ~ 0
 MotorL_Reverce_Out
-Wire Wire Line
-	9300 1100 9450 1100
-Connection ~ 9450 1100
-Wire Wire Line
-	9450 1100 9700 1100
-Connection ~ 9450 2050
-Wire Wire Line
-	9450 2050 9700 2050
 Connection ~ 9700 1100
 Wire Wire Line
@@
 Wire Wire Line
 	8850 1100 9050 1100
-Wire Wire Line
-	8850 2050 9450 2050
 $Comp
 L gekko-rescue:GND-power #PWR029
@@
 Wire Wire Line
 	8300 5050 8300 5400
+Text Notes 6150 7250 0    50   ~ 0
+gate_R\n\n
+Wire Wire Line
+	8850 2050 9700 2050
+Wire Wire Line
+	9300 1100 9700 1100
+Wire Wire Line
+	10400 1100 10750 1100
+Wire Wire Line
+	10400 2050 10850 2050
 $EndSCHEMATC

Commit message: RE_patern
Parts:
- removed Q5: IRLML6344TRPBFTR, micro:IRFML8244TRPBF, symbol gekko-rescue:Q_NMOS_GDS-Device
- added Q1: Q_NMOS_GSD, Package_TO_SOT_SMD:SOT-23, symbol Device:Q_NMOS_GSD
Connections:
- net GND: now also U1.14 (GND), Q1.2 (S)
- net at U3.4 (K), U6.4 (K), U7.4 (K)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: now also Q1.3 (D)
- net at R2.1, R3.2: now also Q1.1 (G)
Changed lines of the file:
@@
 	1600 2350 1600 2550
 Wire Wire Line
-	1600 2550 1800 2550
+	1600 2550 1700 2550
 Wire Wire Line
 	1800 2350 1800 2550
@@
 Text GLabel 6000 3200 1    50   Input ~ 0
 MotorR_Foward
-Text GLabel 5050 4600 0    50   Input ~ 0
-MotorL_Reverce
-Text GLabel 5050 4700 0    50   Input ~ 0
-MotorL_Foward
 Text GLabel 4650 7100 0    50   Input ~ 0
 sens_RR
@@
 Wire Wire Line
 	2250 2050 2250 2400
-$Comp
-L gekko-rescue:Q_NMOS_GDS-Device Q5
-U 1 1 5E4C63DC
-P 5850 7250
-F 0 "Q5" H 6055 7296 50  0000 L CNN
-F 1 "IRLML6344TRPBFTR" H 6000 7000 50  0000 L CNN
-F 2 "micro:IRFML8244TRPBF" H 6050 7350 50  0001 C CNN
-F 3 "~" H 5850 7250 50  0001 C CNN
-	1    5850 7250
-	-1   0    0    1
-$EndComp
 Wire Wire Line
 	6150 7250 6100 7250
@@
 Wire Wire Line
 	4950 7350 5400 7350
-Wire Wire Line
-	5400 7350 5400 7050
-Wire Wire Line
-	5400 7050 5750 7050
 Connection ~ 4950 7350
 Wire Wire Line
@@
 Text GLabel 5700 3200 1    50   Input ~ 0
 battery_sw_CE
-Text GLabel 5500 6300 0    50   Input ~ 0
-BATT_SW
 $Comp
 L Device:D_TVS D4
@@
 Wire Wire Line
 	10400 2050 10850 2050
+$Comp
+L Device:Q_NMOS_GSD Q1
+U 1 1 5EA620E0
+P 5850 7250
+F 0 "Q1" H 6055 7204 50  0000 L CNN
+F 1 "Q_NMOS_GSD" H 6055 7295 50  0000 L CNN
+F 2 "Package_TO_SOT_SMD:SOT-23" H 6050 7350 50  0001 C CNN
+F 3 "~" H 5850 7250 50  0001 C CNN
+	1    5850 7250
+	-1   0    0    -1
+$EndComp
+Wire Wire Line
+	5400 6950 5750 6950
+Wire Wire Line
+	5750 6950 5750 7050
+Wire Wire Line
+	5400 6950 5400 7350
+Wire Wire Line
+	1700 2350 1700 2550
+Connection ~ 1700 2550
+Wire Wire Line
+	1700 2550 1800 2550
+Text GLabel 5050 4700 0    50   Input ~ 0
+MotorL_Foward
+Text GLabel 5050 4600 0    50   Input ~ 0
+MotorL_Reverce
 $EndSCHEMATC

Commit message: RE_patern_finish
Changed lines of the file:
@@
 Connection ~ 9600 5050
 Wire Wire Line
-	9600 5050 9600 5200
+	9600 5050 9600 5150
 NoConn ~ 9900 5500
 Wire Wire Line
@@
 	10550 5300 10750 5300
 Wire Wire Line
-	10150 5050 10150 5300
-Wire Wire Line
 	9600 5050 10000 5050
 Wire Wire Line
@@
 Wire Wire Line
 	10000 5900 10050 5900
-Connection ~ 10000 5050
-Wire Wire Line
-	10000 5050 10150 5050
 Text GLabel 5500 5100 3    50   Input ~ 0
 battery_wt
@@
 Text GLabel 5050 4600 0    50   Input ~ 0
 MotorL_Reverce
+Wire Wire Line
+	9600 5150 10150 5150
+Wire Wire Line
+	10150 5150 10150 5300
+Connection ~ 9600 5150
+Wire Wire Line
+	9600 5150 9600 5200
 $EndSCHEMATC

Commit message: For the time being
Connections:
- net +3V3: now also C11.1, U2.24 (VDD)
Changed lines of the file:
@@
 Wire Wire Line
 	9600 5150 9600 5200
+$Comp
+L gekko-rescue:+3.3V-power #PWR?
+U 1 1 5EC37E5C
+P 7100 5200
+F 0 "#PWR?" H 7100 5050 50  0001 C CNN
+F 1 "+3.3V" H 7115 5373 50  0000 C CNN
+F 2 "" H 7100 5200 50  0001 C CNN
+F 3 "" H 7100 5200 50  0001 C CNN
+	1    7100 5200
+	1    0    0    -1
+$EndComp
+Wire Wire Line
+	6650 5200 7100 5200
+Connection ~ 6650 5200
 $EndSCHEMATC
